Commit message: add data collection

File: urdf/food/forked_food.urdf (robot description, URDF)
Before this commit: robot forked food, 1 links, 0 joints
Links:
- link forked food: geometry collision mesh filename=meshes/forked_food.dae scale=0.04 0.04 0.04; visual box size=0.075 0.075 0.075

File: urdf/franka_description/robots/original_franka.urdf (robot description, URDF)
Before this commit: robot panda, 11 links, 10 joints
Links:
- link panda_hand: mass None -> 5
