Commit message: finish implement affordance baselines

File: urdf/ball/BallHLS.urdf (robot description, URDF)
Before this commit: robot ball, 1 links, 0 joints
Links:
- link ball: mass 0.0033333333333333335 -> 0.0001

File: urdf/container/bowl.urdf (robot description, URDF)
Before this commit: robot bowl, 1 links, 0 joints
Links:
- link bowl: mass 0.5 -> 1

File: urdf/franka_description/robots/original_franka.urdf (robot description, URDF)
Before this commit: robot panda, 11 links, 10 joints
Links:
- link panda_hand: mass 5 -> 10
- link panda_link0: mass None -> 10
- link panda_link1: mass None -> 10
- link panda_link2: mass None -> 10
- link panda_link3: mass None -> 10
- link panda_link4: mass None -> 10
- link panda_link5: mass None -> 10
- link panda_link6: mass None -> 10
- link panda_link7: mass None -> 10

File: urdf/grab_tool/spoon.urdf (robot description, URDF)
Before this commit: robot spoon, 2 links, 1 joints
Links:
- link cube_spoon: mass None -> 0.1
- link spoon: mass 0.5 -> 0.05
