Commit message: add dumbwaiter

File: urdf/microwave/mobility.urdf (robot description, URDF)
Before this commit: robot partnet_c3bb5f3c842a6c2d178e7d331e641179, 3 links, 2 joints
Links:
- link link_0: geometry collision mesh filename=textured_objs/original-1.obj; collision mesh filename=textured_objs/original-10.obj
