Commit message: debug dumbwaiter

File: urdf/dumbwaiter/mobility.urdf (robot description, URDF)
Before this commit: robot partnet_c3bb5f3c842a6c2d178e7d331e641179, 3 links, 2 joints
Links:
- link link_0: geometry collision mesh filename=textured_objs/original-1.obj; collision mesh filename=textured_objs/original-10.obj
- link link_1: geometry collision mesh filename=textured_objs/original-2.obj; collision mesh filename=textured_objs/original-4.obj
